Commit message: Support multiple SC ports per rail on the taskboard for phase 1 (#561) (#582)
* Support up to 3 SC ports per rail (6 total) with min-buffer enforcement

* Clean up

* Create new sample config to test multiple ports

* Formatting

* Only modify task_board.urdf.xacro and launch file, revert changes to aic_engine

File: aic_description/urdf/task_board.urdf.xacro (robot description, xacro)
@@ -63,4 +63,22 @@
   <xacro:arg name="sc_port_1_pitch" default="0.0"/>
   <xacro:arg name="sc_port_1_yaw" default="0.0"/>
+  <!-- SC Port 2 (SC_RAIL_0) -->
+  <xacro:arg name="sc_port_2_present" default="false"/>
+  <xacro:arg name="sc_port_2_translation" default="0.0"/>
+  <xacro:arg name="sc_port_2_roll" default="0.0"/>
+  <xacro:arg name="sc_port_2_pitch" default="0.0"/>
+  <xacro:arg name="sc_port_2_yaw" default="0.0"/>
+  <!-- SC Port 3 (SC_RAIL_1) -->
+  <xacro:arg name="sc_port_3_present" default="false"/>
+  <xacro:arg name="sc_port_3_translation" default="0.0"/>
+  <xacro:arg name="sc_port_3_roll" default="0.0"/>
+  <xacro:arg name="sc_port_3_pitch" default="0.0"/>
+  <xacro:arg name="sc_port_3_yaw" default="0.0"/>
+  <!-- SC Port 4 (SC_RAIL_1) -->
+  <xacro:arg name="sc_port_4_present" default="false"/>
+  <xacro:arg name="sc_port_4_translation" default="0.0"/>
+  <xacro:arg name="sc_port_4_roll" default="0.0"/>
+  <xacro:arg name="sc_port_4_pitch" default="0.0"/>
+  <xacro:arg name="sc_port_4_yaw" default="0.0"/>
   <!-- NIC Card Mount 0 -->
   <xacro:arg name="nic_card_mount_0_present" default="false"/>
@@ -154,5 +172,5 @@
     </joint>
   </xacro:if>
-  <!-- SC Port 0 -->
+  <!-- SC Port 0 (SC_RAIL_0, Y=0.0295) -->
   <xacro:if value="$(arg sc_port_0_present)">
     <xacro:sc_port prefix="sc_port_0" pose="${-0.075 + $(arg sc_port_0_translation)} 0.0295 0.0165 ${1.57 + $(arg sc_port_0_roll)} $(arg sc_port_0_pitch) ${1.57 + $(arg sc_port_0_yaw)}"/>
@@ -164,11 +182,41 @@
     </gazebo>
   </xacro:if>
-  <!-- SC Port 1 -->
+  <!-- SC Port 1 (SC_RAIL_0, Y=0.0295) -->
   <xacro:if value="$(arg sc_port_1_present)">
-    <xacro:sc_port prefix="sc_port_1" pose="${-0.075 + $(arg sc_port_1_translation)} 0.0705 0.0165 ${1.57 + $(arg sc_port_1_roll)} $(arg sc_port_1_pitch) ${1.57 + $(arg sc_port_1_yaw)}"/>
+    <xacro:sc_port prefix="sc_port_1" pose="${-0.075 + $(arg sc_port_1_translation)} 0.0295 0.0165 ${1.57 + $(arg sc_port_1_roll)} $(arg sc_port_1_pitch) ${1.57 + $(arg sc_port_1_yaw)}"/>
     <gazebo>
       <joint name="sc_port_1_joint" type="fixed">
         <parent>task_board_base_link</parent>
         <child>sc_port_1::sc_port_link</child>
+      </joint>
+    </gazebo>
+  </xacro:if>
+  <!-- SC Port 2 (SC_RAIL_0, Y=0.0295) -->
+  <xacro:if value="$(arg sc_port_2_present)">
+    <xacro:sc_port prefix="sc_port_2" pose="${-0.075 + $(arg sc_port_2_translation)} 0.0295 0.0165 ${1.57 + $(arg sc_port_2_roll)} $(arg sc_port_2_pitch) ${1.57 + $(arg sc_port_2_yaw)}"/>
+    <gazebo>
+      <joint name="sc_port_2_joint" type="fixed">
+        <parent>task_board_base_link</parent>
+        <child>sc_port_2::sc_port_link</child>
+      </joint>
+    </gazebo>
+  </xacro:if>
+  <!-- SC Port 3 (SC_RAIL_1, Y=0.0705) -->
+  <xacro:if value="$(arg sc_port_3_present)">
+    <xacro:sc_port prefix="sc_port_3" pose="${-0.075 + $(arg sc_port_3_translation)} 0.0705 0.0165 ${1.57 + $(arg sc_port_3_roll)} $(arg sc_port_3_pitch) ${1.57 + $(arg sc_port_3_yaw)}"/>
+    <gazebo>
+      <joint name="sc_port_3_joint" type="fixed">
+        <parent>task_board_base_link</parent>
+        <child>sc_port_3::sc_port_link</child>
+      </joint>
+    </gazebo>
+  </xacro:if>
+  <!-- SC Port 4 (SC_RAIL_1, Y=0.0705) -->
+  <xacro:if value="$(arg sc_port_4_present)">
+    <xacro:sc_port prefix="sc_port_4" pose="${-0.075 + $(arg sc_port_4_translation)} 0.0705 0.0165 ${1.57 + $(arg sc_port_4_roll)} $(arg sc_port_4_pitch) ${1.57 + $(arg sc_port_4_yaw)}"/>
+    <gazebo>
+      <joint name="sc_port_4_joint" type="fixed">
+        <parent>task_board_base_link</parent>
+        <child>sc_port_4::sc_port_link</child>
       </joint>
     </gazebo>
